File: hardware/Coonix/NUC980/NUC980.kicad_pcb (KiCad board)
At the start: 2 copper layers, 95 x 85 mm, 176 parts, among them J1001 Conn_01x05, J1101 Conn_01x02, J201 8P8C_LED_Shielded, J301 USB_A, J302 USB_C_Receptacle, J303 POWER, J501 Micro_SD_Card, J601 Conn_01x10, J701 Debug_UART, J702 JTAG, J801 AC1583, J901 Conn_01x10, Q701 MMBT3904, SW1201 SW_Push, SW1202 SW_Push, SW1203 SW_Push, SW701 RESET, U1001 MAX485E, U1101 SN65HVD232, U201 NUC980DK, U202 IP101GR, U401 W25N01GV, U701 EA3036, Y201 25MHz, Y701 32.768KHz, Y702 12MHz

Commit message: update pcb and add JLC STM pos, bom file
Parts:
- removed R714, R715, R716, R717: NC, Resistor_SMD:R_0603_1608Metric
- removed the REF** at (133.5, 107.6)
- added SW702: SW_DIP_x04, Button_Switch_THT:SW_DIP_SPSTx04_Piano_10.8x11.72mm_W7.62mm_P2.54mm, F.Cu at (108.5, 112.0)
- C1001, C207, C208, C210, C211, C212, C213, C301, C302, C305, C306, C706, C709, C732, C733, C734, C740, C741, D302, FB201, FB202, JP1001, Q701, R1001, R205, R206, R215, R305, R306, R307, R308, R309, R501, R704, R705, R706, R707, R708, R709, R710, R711, R712: moved to B.Cu
- moved C1001 4.31 mm to (123.6, 122.0), turned to 90 degrees
- moved C213 2.15 mm to (138.8, 94.5)
- moved R206 2.14 mm to (137.7, 93.4)
- moved C211 1.79 mm to (140.3, 95.6)
- moved FB202 1.78 mm to (141.7, 97.0)
- moved R708 0.95 mm to (122.0, 82.8)
- moved R205 0.91 mm to (137.4, 91.5)
- moved R707 0.14 mm to (121.0, 84.4)
- turned R705 to 90 degrees
Routing:
- net Net-(SW702-Pad5): track 3.03 -> 51.9 mm, vias 0 -> 4
- net Net-(SW702-Pad6): track 3.40 -> 49.8 mm, vias 0 -> 4
- net Net-(SW702-Pad7): track 4.21 -> 47.4 mm, vias 0 -> 4
- net Net-(SW702-Pad8): track 9.33 -> 46.3 mm, vias 0 -> 4
- net +5V: track 50.5 -> 43.0 mm, vias 5 -> 3
- net GNDD: track 95.0 -> 101.3 mm, vias 85 -> 270
- net +1V2: track 52.8 -> 48.2 mm, vias 3 -> 10
- net /ETH/PHY_DVDD: track 82.0 -> 86.4 mm, vias 8 -> 7
- net +3V3: track 335.9 -> 338.2 mm, vias 16 -> 29
- net /ETH/ETH_RX_CLK: track 4.19 -> 6.38 mm, vias 0 -> 1
- net Net-(C732-Pad2): track 5.74 -> 7.38 mm, vias 0 -> 1
- net Net-(C706-Pad2): track 3.78 -> 5.37 mm
- net /SD0_CLK: track 46.3 -> 47.6 mm, vias 2 -> 3
- net /~RST: track 162.3 -> 163.5 mm, vias 8 -> 11
- net /PE4: track 21.8 -> 22.9 mm, vias 2 -> 3
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- added copper zone on B.Cu, net +1V2
- added copper zone on B.Cu, net +1V8
- added copper zone on B.Cu, net +3V3
- added copper zone on B.Cu, net +5V
- removed copper zone on F.Cu, net +5V
Other:
- board text added: "NUC980 L 20200511 Rev 1.0"
- board text added: "PG0"
- board text added: "PG1"
- board text added: "PG3"
- board text added: "PG5"
- board text removed: "NUC980 L 20200418"
