File: hardware/Coonix/NUC980/NUC980_CORE.sch (KiCad schematic (older format))
At the start: 80 parts, among them J701 Debug_UART, J702 JTAG, Q701 MMBT3904, SW701 RESET, U201 NUC980DK, U701 EA3036, Y701 32.768KHz, Y702 12MHz

Commit message: update pcb and add JLC STM pos, bom file
Parts:
- removed R714, R715, R716, R717: NC, Resistor_SMD:R_0603_1608Metric, symbol Device:R
- added SW702: SW_DIP_x04, Button_Switch_THT:SW_DIP_SPSTx04_Piano_10.8x11.72mm_W7.62mm_P2.54mm, symbol Switch:SW_DIP_x04
Connections:
- net GNDD: now also SW702.1, SW702.2, SW702.3, SW702.4
- net at U201.25 (PG5): now also SW702.8
- net at U201.26 (PG3): now also SW702.7
- net at U201.27 (PG1): now also SW702.6
- net at U201.28 (PG0): now also SW702.5
Other:
- moved on the sheet: R718, R719, R720, R721
Changed lines of the file:
@@
 PF10
 Wire Wire Line
-	4700 5850 4900 5850
-Wire Wire Line
-	4700 5950 4900 5950
-Wire Wire Line
-	4700 6050 4900 6050
-Wire Wire Line
-	4700 6150 4900 6150
-Wire Wire Line
-	4700 6250 4900 6250
-Wire Wire Line
-	4700 6350 4900 6350
-Wire Wire Line
-	4900 6450 4700 6450
-Wire Wire Line
-	4900 6550 4700 6550
+	4700 5850 4750 5850
+Wire Wire Line
+	4700 5950 4750 5950
+Wire Wire Line
+	4700 6050 4750 6050
+Wire Wire Line
+	4700 6150 4750 6150
 $Comp
 L power:GNDD #PWR0137
@@
 Wire Wire Line
 	5650 5850 5650 5950
-Connection ~ 5650 6550
-Wire Wire Line
-	5650 6550 5200 6550
 Connection ~ 5650 5950
 Wire Wire Line
@@
 	5650 6050 5650 6150
 Connection ~ 5650 6150
-Wire Wire Line
-	5650 6150 5650 6250
-Connection ~ 5650 6250
-Wire Wire Line
-	5650 6250 5650 6350
-Connection ~ 5650 6350
-Wire Wire Line
-	5650 6350 5650 6450
-Connection ~ 5650 6450
-Wire Wire Line
-	5650 6450 5650 6550
 $Comp
 L Connector_Generic:Conn_01x08 J702
@@
 	4150 2050 3600 2050
 $Comp
-L Device:R R714
-U 1 1 5EBC7DB3
-P 5050 5850
-F 0 "R714" V 5000 5600 50  0000 C CNN
-F 1 "NC" V 5000 6050 50  0000 C CNN
-F 2 "Resistor_SMD:R_0603_1608Metric" V 4980 5850 50  0001 C CNN
-F 3 "~" H 5050 5850 50  0001 C CNN
-	1    5050 5850
+L Device:R R719
+U 1 1 5EBCFAE4
+P 5050 6400
+F 0 "R719" V 5000 6150 50  0000 C CNN
+F 1 "NC" V 5000 6600 50  0000 C CNN
+F 2 "Resistor_SMD:R_0603_1608Metric" V 4980 6400 50  0001 C CNN
+F 3 "~" H 5050 6400 50  0001 C CNN
+	1    5050 6400
 	0    1    1    0
 $EndComp
-Wire Wire Line
-	5200 5850 5650 5850
-$Comp
-L Device:R R715
-U 1 1 5EBCF424
+$Comp
+L Device:R R720
+U 1 1 5EBCFDE1
+P 5050 6500
+F 0 "R720" V 5000 6250 50  0000 C CNN
+F 1 "NC" V 5000 6700 50  0000 C CNN
+F 2 "Resistor_SMD:R_0603_1608Metric" V 4980 6500 50  0001 C CNN
+F 3 "~" H 5050 6500 50  0001 C CNN
+	1    5050 6500
+	0    1    1    0
+$EndComp
+$Comp
+L Device:R R721
+U 1 1 5EBD022A
+P 5050 6600
+F 0 "R721" V 5000 6350 50  0000 C CNN
+F 1 "NC" V 5000 6800 50  0000 C CNN
+F 2 "Resistor_SMD:R_0603_1608Metric" V 4980 6600 50  0001 C CNN
+F 3 "~" H 5050 6600 50  0001 C CNN
+	1    5050 6600
+	0    1    1    0
+$EndComp
+Wire Wire Line
+	5350 5950 5650 5950
+Wire Wire Line
+	5350 5850 5650 5850
+Wire Wire Line
+	5350 6050 5650 6050
+Wire Wire Line
+	5350 6150 5650 6150
+$Comp
+L Switch:SW_DIP_x04 SW702
+U 1 1 5EBF3D61
 P 5050 5950
-F 0 "R715" V 5000 5700 50  0000 C CNN
-F 1 "NC" V 5000 6150 50  0000 C CNN
-F 2 "Resistor_SMD:R_0603_1608Metric" V 4980 5950 50  0001 C CNN
+F 0 "SW702" H 4750 5700 50  0000 C CNN
+F 1 "SW_DIP_x04" H 4650 5800 50  0000 C CNN
+F 2 "Button_Switch_THT:SW_DIP_SPSTx04_Piano_10.8x11.72mm_W7.62mm_P2.54mm" H 5050 5950 50  0001 C CNN
 F 3 "~" H 5050 5950 50  0001 C CNN
 	1    5050 5950
-	0    1    1    0
-$EndComp
-Wire Wire Line
-	5200 5950 5650 5950
-$Comp
-L Device:R R716
-U 1 1 5EBCF5B9
-P 5050 6050
-F 0 "R716" V 5000 5800 50  0000 C CNN
-F 1 "NC" V 5000 6250 50  0000 C CNN
-F 2 "Resistor_SMD:R_0603_1608Metric" V 4980 6050 50  0001 C CNN
-F 3 "~" H 5050 6050 50  0001 C CNN
-	1    5050 6050
-	0    1    1    0
-$EndComp
-Wire Wire Line
-	5200 6050 5650 6050
-$Comp
-L Device:R R717
-U 1 1 5EBCF7A7
-P 5050 6150
-F 0 "R717" V 5000 5900 50  0000 C CNN
-F 1 "NC" V 5000 6350 50  0000 C CNN
-F 2 "Resistor_SMD:R_0603_1608Metric" V 4980 6150 50  0001 C CNN
-F 3 "~" H 5050 6150 50  0001 C CNN
-	1    5050 6150
-	0    1    1    0
-$EndComp
-Wire Wire Line
-	5200 6150 5650 6150
+	-1   0    0    1
+$EndComp
+Wire Wire Line
+	5650 6150 5650 6300
 $Comp
 L Device:R R718
 U 1 1 5EBCF8F8
-P 5050 6250
-F 0 "R718" V 5000 6000 50  0000 C CNN
-F 1 "NC" V 5000 6450 50  0000 C CNN
-F 2 "Resistor_SMD:R_0603_1608Metric" V 4980 6250 50  0001 C CNN
-F 3 "~" H 5050 6250 50  0001 C CNN
-	1    5050 6250
+P 5050 6300
+F 0 "R718" V 5000 6050 50  0000 C CNN
+F 1 "NC" V 5000 6500 50  0000 C CNN
+F 2 "Resistor_SMD:R_0603_1608Metric" V 4980 6300 50  0001 C CNN
+F 3 "~" H 5050 6300 50  0001 C CNN
+	1    5050 6300
 	0    1    1    0
 $EndComp
 Wire Wire Line
-	5200 6250 5650 6250
-$Comp
-L Device:R R719
-U 1 1 5EBCFAE4
-P 5050 6350
-F 0 "R719" V 5000 6100 50  0000 C CNN
-F 1 "NC" V 5000 6550 50  0000 C CNN
-F 2 "Resistor_SMD:R_0603_1608Metric" V 4980 6350 50  0001 C CNN
-F 3 "~" H 5050 6350 50  0001 C CNN
-	1    5050 6350
-	0    1    1    0
-$EndComp
-Wire Wire Line
-	5200 6350 5650 6350
-$Comp
-L Device:R R720
-U 1 1 5EBCFDE1
-P 5050 6450
-F 0 "R720" V 5000 6200 50  0000 C CNN
-F 1 "NC" V 5000 6650 50  0000 C CNN
-F 2 "Resistor_SMD:R_0603_1608Metric" V 4980 6450 50  0001 C CNN
-F 3 "~" H 5050 6450 50  0001 C CNN
-	1    5050 6450
-	0    1    1    0
-$EndComp
-Wire Wire Line
-	5200 6450 5650 6450
-$Comp
-L Device:R R721
-U 1 1 5EBD022A
-P 5050 6550
-F 0 "R721" V 5000 6300 50  0000 C CNN
-F 1 "NC" V 5000 6750 50  0000 C CNN
-F 2 "Resistor_SMD:R_0603_1608Metric" V 4980 6550 50  0001 C CNN
-F 3 "~" H 5050 6550 50  0001 C CNN
-	1    5050 6550
-	0    1    1    0
-$EndComp
+	4700 6250 4750 6250
+Wire Wire Line
+	4800 6250 4800 6300
+Wire Wire Line
+	4800 6300 4900 6300
+Wire Wire Line
+	4700 6350 4800 6350
+Wire Wire Line
+	4800 6350 4800 6400
+Wire Wire Line
+	4800 6400 4900 6400
+Wire Wire Line
+	4700 6450 4800 6450
+Wire Wire Line
+	4800 6450 4800 6500
+Wire Wire Line
+	4800 6500 4900 6500
+Wire Wire Line
+	4700 6550 4800 6550
+Wire Wire Line
+	4800 6550 4800 6600
+Wire Wire Line
+	4800 6600 4900 6600
+Wire Wire Line
+	5200 6600 5650 6600
+Wire Wire Line
+	5650 6600 5650 6550
+Connection ~ 5650 6550
+Wire Wire Line
+	5200 6500 5650 6500
+Connection ~ 5650 6500
+Wire Wire Line
+	5650 6500 5650 6550
+Wire Wire Line
+	5200 6400 5650 6400
+Connection ~ 5650 6400
+Wire Wire Line
+	5650 6400 5650 6500
+Wire Wire Line
+	5200 6300 5650 6300
+Connection ~ 5650 6300
+Wire Wire Line
+	5650 6300 5650 6400
+Connection ~ 4750 6250
+Wire Wire Line
+	4750 6250 4800 6250
 $EndSCHEMATC
